Commit message: add cbf clf qp

File: rotors_description/urdf/pelican_with_rgbd.xacro (robot description, xacro)
@@ -57,5 +57,5 @@
     enable_depth="true"
     enable_ground_truth="false">
-    <origin xyz="0.1 0.0 -0.03" rpy="0.0 0.0 0.0" />
+    <origin xyz="0.0 0.0 0.1" rpy="0.0 0.0 0.0" />
   </xacro:vi_sensor_macro>
 </robot>
